File: PPGv2.sch (EAGLE design)
At the start: 54 parts

Commit message: Final
-removed extra connectors
-without IR-INP input
Parts:
- removed +12V, -12V, FILTER, INVERTOUT, IR-INP, LEDGND, OUT1: (no value), jumper:JP1E
- removed GND, GND2, LEDS, VOUT(DC): (no value), jumper:JP2E
- removed R2, R27, R3, R4: (no value), resistor:R-US_R0603
Connections:
- removed net N$2 (its old number): IR-INP.2, R4.2
- removed net N$28: LEDS.3, R2.1
- removed net N$3: LEDS.1, R3.1
- removed net N$30: LEDGND.2, R3.2
- removed net N$33: LEDGND.1, R2.2
- removed net N$4: R27.2, R4.1, U$1A.IN-
- removed net N$5: INVERTOUT.1, INVERTOUT.2, R27.1, U$1A.OUT
- net +12V: now also VOUT(AC).2; no longer +12V.1, +12V.2, LEDS.2
- net -12V: now also VOUT(AC).3; no longer -12V.1, -12V.2
- net GND: no longer GND.1, GND.2, GND.3, GND2.1, GND2.2, GND2.3, U$1A.IN+
- net N$18: no longer FILTER.1, FILTER.2
- net N$20: no longer VOUT(AC).2, VOUT(AC).3
- net N$22: no longer OUT1.1, OUT1.2
- net N$29: no longer VOUT(DC).1, VOUT(DC).3

Commit message: -final
Other:
- note added: "Can use this for IR-INP in furture"
Changed lines of the file:
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@@
 <text x="45.72" y="-2.54" size="1.778" layer="92">O/P will be same as I/P</text>
 <text x="-25.4" y="38.1" size="1.778" layer="92">Non-Inverting amplifier</text>
+<text x="-180.34" y="119.38" size="1.778" layer="91">Can use this for IR-INP in furture</text>
 </plain>
 <instances>

Commit message: -final iteration
Other:
- note added: "active LPF"
Changed lines of the file:
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@@
 <text x="-25.4" y="38.1" size="1.778" layer="92">Non-Inverting amplifier</text>
 <text x="-180.34" y="119.38" size="1.778" layer="91">Can use this for IR-INP in furture</text>
+<circle x="175.26" y="45.72" radius="35.28680625" width="0.1524" layer="91"/>
+<text x="170.18" y="71.12" size="1.778" layer="91">active LPF</text>
+<wire x1="63.5" y1="111.76" x2="88.9" y2="111.76" width="0.1524" layer="98"/>
+<wire x1="88.9" y1="111.76" x2="88.9" y2="119.38" width="0.1524" layer="98"/>
+<wire x1="88.9" y1="119.38" x2="111.76" y2="119.38" width="0.1524" layer="98"/>
+<wire x1="111.76" y1="119.38" x2="111.76" y2="93.98" width="0.1524" layer="98"/>
 </plain>
 <instances>
@@
 </segment>
 </net>
+<net name="N$3" class="0">
+<segment>
+<wire x1="76.2" y1="83.82" x2="43.18" y2="83.82" width="0.1524" layer="91"/>
+<wire x1="43.18" y1="83.82" x2="43.18" y2="81.28" width="0.1524" layer="91"/>
+<wire x1="43.18" y1="81.28" x2="88.9" y2="81.28" width="0.1524" layer="91"/>
+<wire x1="88.9" y1="81.28" x2="88.9" y2="99.06" width="0.1524" layer="91"/>
+</segment>
+</net>
